Commit message: cpp joint controller

File: snakebot/urdf/snakebot.urdf (robot description, URDF)
Before this commit: robot snakebot, 8 links, 7 joints
Joints:
- joint joint_1: limit lower=-0.45 upper=0.45 effort=1000 velocity=1.0 -> lower=-1.0 upper=1.0 effort=1000 velocity=1.0
- joint joint_2: limit lower=-0.45 upper=0.45 effort=1000 velocity=1.0 -> lower=-1.0 upper=1.0 effort=1000 velocity=1.0
- joint joint_3: limit lower=-0.45 upper=0.45 effort=1000 velocity=1.0 -> lower=-1.0 upper=1.0 effort=1000 velocity=1.0
- joint joint_4: limit lower=-0.45 upper=0.45 effort=1000 velocity=1.0 -> lower=-1.0 upper=1.0 effort=1000 velocity=1.0
- joint joint_5: limit lower=-0.45 upper=0.45 effort=1000 velocity=1.0 -> lower=-1.0 upper=1.0 effort=1000 velocity=1.0
- joint joint_6: limit lower=-0.45 upper=0.45 effort=1000 velocity=1.0 -> lower=-1.0 upper=1.0 effort=1000 velocity=1.0
- joint joint_7: limit lower=-0.45 upper=0.45 effort=1000 velocity=1.0 -> lower=-1.0 upper=1.0 effort=1000 velocity=1.0
